Commit message: 0925

File: legged_gym/resources/robots/T1_skate/urdf/T1_serial.urdf (robot description, URDF)
Before this commit: robot T1, 24 links, 23 joints
Links:
- link AL1: geometry visual mesh filename=../meshes/AL1.STL
- link AL2: geometry visual mesh filename=../meshes/AL2.STL
- link AL3: geometry collision cylinder length=0.15 radius=0.03; visual mesh filename=../meshes/AL3.STL
- link AR1: geometry visual mesh filename=../meshes/AR1.STL
- link AR2: geometry visual mesh filename=../meshes/AR2.STL
- link AR3: geometry collision cylinder length=0.15 radius=0.03; visual mesh filename=../meshes/AR3.STL
- link Ankle_Cross_Left: geometry visual mesh filename=../meshes/Ankle_Cross_Left.STL
- link Ankle_Cross_Right: geometry visual mesh filename=../meshes/Ankle_Cross_Right.STL
- link H1: geometry visual mesh filename=../meshes/H1.STL
- link H2: geometry collision sphere radius=0.08; visual mesh filename=../meshes/H2.STL
- link Hip_Pitch_Left: geometry visual mesh filename=../meshes/Hip_Pitch_Left.STL
- link Hip_Pitch_Right: geometry visual mesh filename=../meshes/Hip_Pitch_Right.STL
- link Hip_Roll_Left: geometry visual mesh filename=../meshes/Hip_Roll_Left.STL
- link Hip_Roll_Right: geometry visual mesh filename=../meshes/Hip_Roll_Right.STL
- link Hip_Yaw_Left: geometry collision cylinder length=0.16 radius=0.05; visual mesh filename=../meshes/Hip_Yaw_Left.STL
- link Hip_Yaw_Right: geometry collision cylinder length=0.16 radius=0.05; visual mesh filename=../meshes/Hip_Yaw_Right.STL
- link Shank_Left: geometry collision cylinder length=0.15 radius=0.05; visual mesh filename=../meshes/Shank_Left.STL
- link Shank_Right: geometry collision cylinder length=0.15 radius=0.05; visual mesh filename=../meshes/Shank_Right.STL
- link Trunk: geometry collision box size=0.15 0.2 0.3; visual mesh filename=../meshes/Trunk.STL
- link Waist: geometry visual mesh filename=../meshes/Waist.STL
- link left_foot_link: geometry collision box size=0.223 0.1 0.03; visual mesh filename=../meshes/left_foot_link.STL
- link left_hand_link: geometry collision cylinder length=0.175 radius=0.03; visual mesh filename=../meshes/left_hand_link.STL
- link right_foot_link: geometry collision box size=0.223 0.1 0.03; visual mesh filename=../meshes/right_foot_link.STL
- link right_hand_link: geometry collision cylinder length=0.175 radius=0.03; visual mesh filename=../meshes/right_hand_link.STL
